File: thumbler.sch (KiCad schematic (older format))
At the start: 253 parts, among them J1 Conn_01x04, J2 DIN-5_180degree, J3 USB_B_Micro, J4 Conn_01x04, J5 USB_B_Micro, J6 Conn_01x04, J7 DIN-5_180degree, J8 Conn_01x04, SW1 SW_Push, SW2 SW_DIP_x05, SW3 SW_Push, SW4 SW_DIP_x05, U1 MCP1700-3302E_SOT89, U2 STM32F072C8Tx, U3 MCP1700-3302E_SOT89, U4 STM32F072C8Tx, X1 ENCODER_ANO

Commit message: layout wip
Parts:
- C10, C15, C16, C17, C18, C19, C20, C21, C3, C4, C5, C6, C7, C8: footprint Capacitor_SMD:C_0805_2012Metric_Pad1.18x1.45mm_HandSolder -> Capacitor_SMD:C_0603_1608Metric_Pad1.08x0.95mm_HandSolder
Other:
- note added: "Break out encoder and mount on plate?"
Changed lines of the file:
@@
 F 0 "C4" H 5292 4296 50  0000 L CNN
 F 1 "4u7" H 5292 4205 50  0000 L CNN
-F 2 "Capacitor_SMD:C_0805_2012Metric_Pad1.18x1.45mm_HandSolder" H 5200 4250 50  0001 C CNN
+F 2 "Capacitor_SMD:C_0603_1608Metric_Pad1.08x0.95mm_HandSolder" H 5200 4250 50  0001 C CNN
 F 3 "~" H 5200 4250 50  0001 C CNN
 	1    5200 4250
@@
 F 0 "C5" H 5642 4296 50  0000 L CNN
 F 1 "100n" H 5642 4205 50  0000 L CNN
-F 2 "Capacitor_SMD:C_0805_2012Metric_Pad1.18x1.45mm_HandSolder" H 5550 4250 50  0001 C CNN
+F 2 "Capacitor_SMD:C_0603_1608Metric_Pad1.08x0.95mm_HandSolder" H 5550 4250 50  0001 C CNN
 F 3 "~" H 5550 4250 50  0001 C CNN
 	1    5550 4250
@@
 F 0 "C6" H 5992 4296 50  0000 L CNN
 F 1 "100n" H 5992 4205 50  0000 L CNN
-F 2 "Capacitor_SMD:C_0805_2012Metric_Pad1.18x1.45mm_HandSolder" H 5900 4250 50  0001 C CNN
+F 2 "Capacitor_SMD:C_0603_1608Metric_Pad1.08x0.95mm_HandSolder" H 5900 4250 50  0001 C CNN
 F 3 "~" H 5900 4250 50  0001 C CNN
 	1    5900 4250
@@
 F 0 "C7" H 6342 4296 50  0000 L CNN
 F 1 "100n" H 6342 4205 50  0000 L CNN
-F 2 "Capacitor_SMD:C_0805_2012Metric_Pad1.18x1.45mm_HandSolder" H 6250 4250 50  0001 C CNN
+F 2 "Capacitor_SMD:C_0603_1608Metric_Pad1.08x0.95mm_HandSolder" H 6250 4250 50  0001 C CNN
 F 3 "~" H 6250 4250 50  0001 C CNN
 	1    6250 4250
@@
 F 0 "C3" H 4942 4296 50  0000 L CNN
 F 1 "4u7" H 4942 4205 50  0000 L CNN
-F 2 "Capacitor_SMD:C_0805_2012Metric_Pad1.18x1.45mm_HandSolder" H 4850 4250 50  0001 C CNN
+F 2 "Capacitor_SMD:C_0603_1608Metric_Pad1.08x0.95mm_HandSolder" H 4850 4250 50  0001 C CNN
 F 3 "~" H 4850 4250 50  0001 C CNN
 	1    4850 4250
@@
 F 0 "C8" H 6692 4296 50  0000 L CNN
 F 1 "1u" H 6692 4205 50  0000 L CNN
-F 2 "Capacitor_SMD:C_0805_2012Metric_Pad1.18x1.45mm_HandSolder" H 6600 4250 50  0001 C CNN
+F 2 "Capacitor_SMD:C_0603_1608Metric_Pad1.08x0.95mm_HandSolder" H 6600 4250 50  0001 C CNN
 F 3 "~" H 6600 4250 50  0001 C CNN
 	1    6600 4250
@@
 F 0 "C10" H 6992 4296 50  0000 L CNN
 F 1 "10n" H 6992 4205 50  0000 L CNN
-F 2 "Capacitor_SMD:C_0805_2012Metric_Pad1.18x1.45mm_HandSolder" H 6900 4250 50  0001 C CNN
+F 2 "Capacitor_SMD:C_0603_1608Metric_Pad1.08x0.95mm_HandSolder" H 6900 4250 50  0001 C CNN
 F 3 "~" H 6900 4250 50  0001 C CNN
 	1    6900 4250
@@
 F 0 "C16" H 20192 4296 50  0000 L CNN
 F 1 "4u7" H 20192 4205 50  0000 L CNN
-F 2 "Capacitor_SMD:C_0805_2012Metric_Pad1.18x1.45mm_HandSolder" H 20100 4250 50  0001 C CNN
+F 2 "Capacitor_SMD:C_0603_1608Metric_Pad1.08x0.95mm_HandSolder" H 20100 4250 50  0001 C CNN
 F 3 "~" H 20100 4250 50  0001 C CNN
 	1    20100 4250
@@
 F 0 "C17" H 20542 4296 50  0000 L CNN
 F 1 "100n" H 20542 4205 50  0000 L CNN
-F 2 "Capacitor_SMD:C_0805_2012Metric_Pad1.18x1.45mm_HandSolder" H 20450 4250 50  0001 C CNN
+F 2 "Capacitor_SMD:C_0603_1608Metric_Pad1.08x0.95mm_HandSolder" H 20450 4250 50  0001 C CNN
 F 3 "~" H 20450 4250 50  0001 C CNN
 	1    20450 4250
@@
 F 0 "C18" H 20892 4296 50  0000 L CNN
 F 1 "100n" H 20892 4205 50  0000 L CNN
-F 2 "Capacitor_SMD:C_0805_2012Metric_Pad1.18x1.45mm_HandSolder" H 20800 4250 50  0001 C CNN
+F 2 "Capacitor_SMD:C_0603_1608Metric_Pad1.08x0.95mm_HandSolder" H 20800 4250 50  0001 C CNN
 F 3 "~" H 20800 4250 50  0001 C CNN
 	1    20800 4250
@@
 F 0 "C19" H 21242 4296 50  0000 L CNN
 F 1 "100n" H 21242 4205 50  0000 L CNN
-F 2 "Capacitor_SMD:C_0805_2012Metric_Pad1.18x1.45mm_HandSolder" H 21150 4250 50  0001 C CNN
+F 2 "Capacitor_SMD:C_0603_1608Metric_Pad1.08x0.95mm_HandSolder" H 21150 4250 50  0001 C CNN
 F 3 "~" H 21150 4250 50  0001 C CNN
 	1    21150 4250
@@
 F 0 "C15" H 19842 4296 50  0000 L CNN
 F 1 "4u7" H 19842 4205 50  0000 L CNN
-F 2 "Capacitor_SMD:C_0805_2012Metric_Pad1.18x1.45mm_HandSolder" H 19750 4250 50  0001 C CNN
+F 2 "Capacitor_SMD:C_0603_1608Metric_Pad1.08x0.95mm_HandSolder" H 19750 4250 50  0001 C CNN
 F 3 "~" H 19750 4250 50  0001 C CNN
 	1    19750 4250
@@
 F 0 "C20" H 21592 4296 50  0000 L CNN
 F 1 "1u" H 21592 4205 50  0000 L CNN
-F 2 "Capacitor_SMD:C_0805_2012Metric_Pad1.18x1.45mm_HandSolder" H 21500 4250 50  0001 C CNN
+F 2 "Capacitor_SMD:C_0603_1608Metric_Pad1.08x0.95mm_HandSolder" H 21500 4250 50  0001 C CNN
 F 3 "~" H 21500 4250 50  0001 C CNN
 	1    21500 4250
@@
 F 0 "C21" H 21892 4296 50  0000 L CNN
 F 1 "10n" H 21892 4205 50  0000 L CNN
-F 2 "Capacitor_SMD:C_0805_2012Metric_Pad1.18x1.45mm_HandSolder" H 21800 4250 50  0001 C CNN
+F 2 "Capacitor_SMD:C_0603_1608Metric_Pad1.08x0.95mm_HandSolder" H 21800 4250 50  0001 C CNN
 F 3 "~" H 21800 4250 50  0001 C CNN
 	1    21800 4250
@@
 NoConn ~ 20250 6750
 NoConn ~ 20250 6650
+Text Notes 9250 11650 1    50   ~ 0
+Break out encoder and mount on plate?
 $EndSCHEMATC

Commit message: left side re-layout mostly done
Parts:
- removed D30: 1N4148, Diode_THT:D_DO-35_SOD27_P7.62mm_Horizontal, symbol Diode:1N4148
- removed S30: Kailh_Hotplug, keyswitches:Kailh_socket_MX_platemount, symbol kailh_hotplug_mx_plate:Kailh_Hotplug
- added D73, D74: 1N4148, Diode_THT:D_DO-35_SOD27_P7.62mm_Horizontal, symbol Diode:1N4148
- added S68, S69: Kailh_Hotplug, keyswitches:Kailh_socket_MX_platemount, symbol kailh_hotplug_mx_plate:Kailh_Hotplug
- renumbered C22 to C13, C13 to C14, C14 to C15, C15 to C16, C16 to C17, C17 to C18, C18 to C19, C19 to C20, C20 to C21, C21 to C22, C9 to C4, C4 to C5, C5 to C6, C6 to C7, C7 to C8, C8 to C9, D74 to D1, D21 to D10, D22 to D11, D23 to D12, D24 to D13, D15 to D14, D16 to D15, D17 to D16, D18 to D17, D19 to D18, D10 to D19, D63 to D2, D11 to D20, D12 to D21, D13 to D22, D14 to D23, D5 to D24, D6 to D25, D7 to D26, D8 to D27, D9 to D28, D64 to D29, D31 to D3, D65 to D30, D66 to D31, D1 to D32, D2 to D33, D3 to D34, D4 to D35, D59 to D36, D60 to D37, D61 to D38, D62 to D39, D28 to D4, D54 to D40, D55 to D41, D56 to D42, D57 to D43, D58 to D44, D68 to D45, D49 to D46, D50 to D47, D51 to D48, D52 to D49, D29 to D5, D53 to D50, D72 to D51, D69 to D52, D70 to D53, D71 to D54, D73 to D55, D44 to D56, D45 to D57, D46 to D58, D47 to D59, D25 to D6, D48 to D60, D39 to D61, D40 to D62, D41 to D63, D42 to D64, D43 to D65, D75 to D66, D36 to D67, D37 to D68, D34 to D69, D26 to D7, D35 to D70, D38 to D71, D32 to D72, D33 to D75, D67 to D76, D27 to D8, D20 to D9, J5 to J1, J1 to J2, J6 to J3, J2 to J4, J4 to J5, J7 to J6, J8 to J7, J3 to J8, R3 to R1, R13 to R10, R14 to R11, R15 to R12, R17 to R13, R20 to R14, R18 to R15, R19 to R16, R21 to R17, R23 to R18, R22 to R19, R5 to R2, R24 to R20, R6 to R21, R7 to R22, R25 to R23, R26 to R24, R27 to R25, R28 to R26, R8 to R27, R1 to R3, R9 to R5, R10 to R6, R2 to R7, R11 to R8, R12 to R9, S31 to S1, S23 to S10, S24 to S11, S15 to S12, S16 to S13, S17 to S14, S18 to S15, S19 to S16, S10 to S17, S11 to S18, S12 to S19, S28 to S2, S13 to S20, S14 to S21, S5 to S22, S6 to S23, S7 to S24, S8 to S25, S9 to S26, S63 to S27, S64 to S28, S65 to S29, S29 to S3, S1 to S30, S2 to S31, S3 to S32, S4 to S33, S66 to S34, S59 to S35, S60 to S36, S61 to S37, S62 to S38, S54 to S39, S25 to S4, S55 to S40, S56 to S41, S57 to S42, S58 to S43, S67 to S44, S68 to S45, S69 to S46, S49 to S47, S50 to S48, S51 to S49, S26 to S5, S52 to S50, S53 to S51, S44 to S52, S45 to S53, S46 to S54, S47 to S55, S48 to S56, S39 to S57, S40 to S58, S41 to S59, S27 to S6, S42 to S60, S43 to S61, S36 to S62, S37 to S63, S34 to S64, S35 to S65, S38 to S66, S32 to S67, S20 to S7, S33 to S70, S21 to S8, S22 to S9, TP37 to TP1, TP8 to TP10, TP9 to TP11, TP10 to TP12, TP11 to TP13, TP12 to TP14, TP14 to TP15, TP15 to TP16, TP16 to TP17, TP17 to TP18, TP18 to TP19, TP1 to TP2, TP19 to TP20, TP20 to TP21, TP38 to TP22, TP21 to TP23, TP22 to TP24, TP23 to TP25, TP24 to TP26, TP25 to TP27, TP26 to TP28, TP27 to TP29, TP2 to TP3, TP28 to TP30, TP29 to TP31, TP30 to TP32, TP31 to TP33, TP32 to TP34, TP33 to TP35, TP34 to TP36, TP35 to TP37, TP36 to TP38, TP3 to TP4, TP4 to TP5, TP5 to TP6, TP6 to TP7, TP7 to TP8, TP13 to TP9, U2 to U1, U1 to U2
Connections:
- net R_ROW3: now also D73.1 (K)
- net R_ROW4: now also D74.1 (K)
- net at R25.2, S62.2, S63.2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: now also S64.2, S65.2
- net at R26.2, S67.2, S70.2: now also S68.2, S69.2; no longer S64.2, S65.2
- new net: D73.2 (A), S68.1
- new net: D74.2 (A), S69.1
Other:
- moved on the sheet: D69, D70, S64, S65
