File: thumbler.kicad_pcb (KiCad board)
At the start: 2 copper layers, 257 parts, among them J1 USB_B_Micro, J2 Conn_01x04, J3 Conn_01x04, J4 DIN-5_180degree, J5 Conn_01x04, J6 DIN-5_180degree, J7 Conn_01x04, J8 USB_B_Micro, SW1 SW_Push, SW2 SW_DIP_x05, SW3 SW_Push, SW4 SW_DIP_x05, U1 STM32F072C8Tx, U2 MCP1700-3302E_SOT89, U3 MCP1700-3302E_SOT89, U4 STM32F072C8Tx, X1 ENCODER_ANO

Commit message: 70 key laid out
Parts:
- removed the D36 at (352.8, 261.9)
- removed the S35 at (361.7, 253.8)
- added D77: RED, LED_SMD:LED_1206_3216Metric_Pad1.42x1.75mm_HandSolder, B.Cu at (458.1, 135.5)
- added S71: Kailh_Hotplug, keyswitches:Kailh_socket_MX_platemount, F.Cu at (466.5, 257.8)
- D76: value RED -> 1N4148; footprint LED_SMD:LED_1206_3216Metric_Pad1.42x1.75mm_HandSolder -> Diode_THT:D_DO-35_SOD27_P7.62mm_Horizontal; moved to F.Cu
- moved TP17 191.0 mm to (75.9, 246.6)
- moved TP20 191.0 mm to (66.4, 243.0)
- moved TP15 191.0 mm to (66.3, 247.8)
- moved TP16 191.0 mm to (70.2, 243.9)
- moved TP18 191.0 mm to (61.3, 242.7)
- moved TP19 191.0 mm to (71.5, 247.1)
- moved TP21 191.0 mm to (61.9, 246.7)
- moved S34 162.1 mm to (326.7, 322.9)
- moved D76 130.2 mm to (457.6, 265.8)
- moved X1 100.7 mm to (196.4, 287.9)
- moved D29 47.3 mm to (244.5, 269.1)
- moved S28 47.3 mm to (264.7, 282.8)
- moved TP9 47.3 mm to (256.8, 250.8)
- moved R11 47.3 mm to (259.8, 249.9)
- moved D30 47.3 mm to (255.7, 290.8)
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- renumbered D36 to D37, D36 to D38, D36 to D39, D36 to D40, D36 to D41, D36 to D42, D36 to D43, D36 to D44, D36 to D46, D36 to D47, D36 to D48, D36 to D49, D36 to D50, D36 to D56, D36 to D57, D36 to D58, D36 to D59, D36 to D60, D36 to D61, D36 to D62, D36 to D63, D36 to D64, D36 to D65, D36 to D67, D36 to D68, D36 to D69, D36 to D70, D36 to D71, D36 to D72, D36 to D73, D36 to D74, D36 to D75, S35 to S36, S35 to S37, S35 to S38, S35 to S39, S35 to S40, S35 to S41, S35 to S42, S35 to S43, S35 to S47, S35 to S48, S35 to S49, S35 to S50, S35 to S51, S35 to S52, S35 to S53, S35 to S54, S35 to S55, S35 to S56, S35 to S57, S35 to S58, S35 to S59, S35 to S60, S35 to S61, S35 to S62, S35 to S63, S35 to S64, S35 to S65, S35 to S66, S35 to S67, S35 to S68, S35 to S69, S35 to S70
Connections:
- D76 pad 1: Net-(D76-Pad1) -> R_ROW5
- D76 pad 2: +3V3 -> Net-(D76-Pad2)
- R27 pad 1: Net-(D76-Pad1) -> Net-(D77-Pad1)
Routing:
- net Net-(D36-Pad2): track 121.6 -> 118.1 mm
- net Net-(D76-Pad2): track 0.00 -> 3.48 mm

Commit message: all TPs to front
Parts:
- TP10, TP11, TP12, TP13, TP14, TP15, TP16, TP17, TP18, TP19, TP2, TP20, TP21, TP23, TP24, TP25, TP26, TP27, TP28, TP29, TP3, TP30, TP31, TP32, TP33, TP34, TP35, TP36, TP37, TP38, TP4, TP5, TP6, TP7, TP8, TP9: moved to F.Cu
- moved R26 177.3 mm to (486.1, 156.9), turned to 270 degrees
- moved R25 145.6 mm to (457.1, 156.9), turned to 270 degrees
- moved R15 105.3 mm to (387.3, 163.2), turned to 270 degrees
- moved TP18 104.1 mm to (157.6, 282.3)
- moved TP20 103.9 mm to (162.6, 282.0)
- moved TP16 103.2 mm to (166.5, 281.1)
- moved TP21 101.4 mm to (158.2, 278.4)
- moved TP19 101.1 mm to (167.7, 278.0)
- moved TP15 100.7 mm to (162.6, 277.3)
- moved TP17 100.6 mm to (172.6, 274.2)
- moved R13 60.8 mm to (316.5, 168.0)
- moved R16 60.8 mm to (338.2, 168.9)
- moved R19 60.8 mm to (316.0, 178.7)
- moved R20 60.8 mm to (324.4, 170.8)
- moved R24 60.8 mm to (335.9, 176.8)
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Connections:
- D37 pad 1: R_ROW2 -> R_ROW3
- D37 pad 2: Net-(D36-Pad2) -> Net-(D37-Pad2)
- D38 pad 1: R_ROW2 -> R_ROW4
- D38 pad 2: Net-(D36-Pad2) -> Net-(D38-Pad2)
- D39 pad 1: R_ROW2 -> R_ROW5
- D39 pad 2: Net-(D36-Pad2) -> Net-(D39-Pad2)
- D40 pad 1: R_ROW2 -> R_ROW1
- D40 pad 2: Net-(D36-Pad2) -> Net-(D40-Pad2)
- D41 pad 2: Net-(D36-Pad2) -> Net-(D41-Pad2)
- D42 pad 1: R_ROW2 -> R_ROW3
- D42 pad 2: Net-(D36-Pad2) -> Net-(D42-Pad2)
- D43 pad 1: R_ROW2 -> R_ROW4
- D43 pad 2: Net-(D36-Pad2) -> Net-(D43-Pad2)
- D44 pad 1: R_ROW2 -> R_ROW5
- D44 pad 2: Net-(D36-Pad2) -> Net-(D44-Pad2)
- D46 pad 1: R_ROW2 -> R_ROW1
- D46 pad 2: Net-(D36-Pad2) -> Net-(D46-Pad2)
- D47 pad 2: Net-(D36-Pad2) -> Net-(D47-Pad2)
- D48 pad 1: R_ROW2 -> R_ROW3
- D48 pad 2: Net-(D36-Pad2) -> Net-(D48-Pad2)
- D49 pad 1: R_ROW2 -> R_ROW4
- D49 pad 2: Net-(D36-Pad2) -> Net-(D49-Pad2)
- D50 pad 1: R_ROW2 -> R_ROW5
- D50 pad 2: Net-(D36-Pad2) -> Net-(D50-Pad2)
- D56 pad 1: R_ROW2 -> R_ROW1
- D56 pad 2: Net-(D36-Pad2) -> Net-(D56-Pad2)
- D57 pad 2: Net-(D36-Pad2) -> Net-(D57-Pad2)
- D58 pad 1: R_ROW2 -> R_ROW3
- D58 pad 2: Net-(D36-Pad2) -> Net-(D58-Pad2)
- D59 pad 1: R_ROW2 -> R_ROW4
- D59 pad 2: Net-(D36-Pad2) -> Net-(D59-Pad2)
- D60 pad 1: R_ROW2 -> R_ROW5
- D60 pad 2: Net-(D36-Pad2) -> Net-(D60-Pad2)
- D61 pad 1: R_ROW2 -> R_ROW1
- D61 pad 2: Net-(D36-Pad2) -> Net-(D61-Pad2)
- D62 pad 2: Net-(D36-Pad2) -> Net-(D62-Pad2)
- D63 pad 1: R_ROW2 -> R_ROW3
- D63 pad 2: Net-(D36-Pad2) -> Net-(D63-Pad2)
- D64 pad 1: R_ROW2 -> R_ROW4
- D64 pad 2: Net-(D36-Pad2) -> Net-(D64-Pad2)
- D65 pad 1: R_ROW2 -> R_ROW5
- D65 pad 2: Net-(D36-Pad2) -> Net-(D65-Pad2)
- D67 pad 1: R_ROW2 -> R_ROW1
- D67 pad 2: Net-(D36-Pad2) -> Net-(D67-Pad2)
- D68 pad 2: Net-(D36-Pad2) -> Net-(D68-Pad2)
- D69 pad 1: R_ROW2 -> R_ROW3
- D69 pad 2: Net-(D36-Pad2) -> Net-(D69-Pad2)
- D70 pad 1: R_ROW2 -> R_ROW4
- D70 pad 2: Net-(D36-Pad2) -> Net-(D70-Pad2)
- D71 pad 1: R_ROW2 -> R_ROW5
- D71 pad 2: Net-(D36-Pad2) -> Net-(D71-Pad2)
- D72 pad 1: R_ROW2 -> R_ROW1
- D72 pad 2: Net-(D36-Pad2) -> Net-(D72-Pad2)
- D73 pad 2: Net-(D36-Pad2) -> Net-(D73-Pad2)
- D74 pad 1: R_ROW2 -> R_ROW3
- D74 pad 2: Net-(D36-Pad2) -> Net-(D74-Pad2)
- D75 pad 1: R_ROW2 -> R_ROW4
- D75 pad 2: Net-(D36-Pad2) -> Net-(D75-Pad2)
- S36 pad 1: Net-(D36-Pad2) -> Net-(D37-Pad2)
- S37 pad 1: Net-(D36-Pad2) -> Net-(D38-Pad2)
- S38 pad 1: Net-(D36-Pad2) -> Net-(D39-Pad2)
- S39 pad 1: Net-(D36-Pad2) -> Net-(D40-Pad2)
- S39 pad 2: Net-(R13-Pad2) -> Net-(R15-Pad2)
- S40 pad 1: Net-(D36-Pad2) -> Net-(D41-Pad2)
- S40 pad 2: Net-(R13-Pad2) -> Net-(R15-Pad2)
- S41 pad 1: Net-(D36-Pad2) -> Net-(D42-Pad2)
- S41 pad 2: Net-(R13-Pad2) -> Net-(R15-Pad2)
- S42 pad 1: Net-(D36-Pad2) -> Net-(D43-Pad2)
- S42 pad 2: Net-(R13-Pad2) -> Net-(R15-Pad2)
- S43 pad 1: Net-(D36-Pad2) -> Net-(D44-Pad2)
- S43 pad 2: Net-(R13-Pad2) -> Net-(R15-Pad2)
- S47 pad 1: Net-(D36-Pad2) -> Net-(D46-Pad2)
- S47 pad 2: Net-(R13-Pad2) -> Net-(R19-Pad2)
- S48 pad 1: Net-(D36-Pad2) -> Net-(D47-Pad2)
- S48 pad 2: Net-(R13-Pad2) -> Net-(R19-Pad2)
- S49 pad 1: Net-(D36-Pad2) -> Net-(D48-Pad2)
- S49 pad 2: Net-(R13-Pad2) -> Net-(R19-Pad2)
- S50 pad 1: Net-(D36-Pad2) -> Net-(D49-Pad2)
- S50 pad 2: Net-(R13-Pad2) -> Net-(R19-Pad2)
- S51 pad 1: Net-(D36-Pad2) -> Net-(D50-Pad2)
- S51 pad 2: Net-(R13-Pad2) -> Net-(R19-Pad2)
- S52 pad 1: Net-(D36-Pad2) -> Net-(D56-Pad2)
- S52 pad 2: Net-(R13-Pad2) -> Net-(R20-Pad2)
- S53 pad 1: Net-(D36-Pad2) -> Net-(D57-Pad2)
- S53 pad 2: Net-(R13-Pad2) -> Net-(R20-Pad2)
- S54 pad 1: Net-(D36-Pad2) -> Net-(D58-Pad2)
- S54 pad 2: Net-(R13-Pad2) -> Net-(R20-Pad2)
- S55 pad 1: Net-(D36-Pad2) -> Net-(D59-Pad2)
- S55 pad 2: Net-(R13-Pad2) -> Net-(R20-Pad2)
- S56 pad 1: Net-(D36-Pad2) -> Net-(D60-Pad2)
- S56 pad 2: Net-(R13-Pad2) -> Net-(R20-Pad2)
- S57 pad 1: Net-(D36-Pad2) -> Net-(D61-Pad2)
- S57 pad 2: Net-(R13-Pad2) -> Net-(R24-Pad2)
- S58 pad 1: Net-(D36-Pad2) -> Net-(D62-Pad2)
- S58 pad 2: Net-(R13-Pad2) -> Net-(R24-Pad2)
- S59 pad 1: Net-(D36-Pad2) -> Net-(D63-Pad2)
- S59 pad 2: Net-(R13-Pad2) -> Net-(R24-Pad2)
- S60 pad 1: Net-(D36-Pad2) -> Net-(D64-Pad2)
- S60 pad 2: Net-(R13-Pad2) -> Net-(R24-Pad2)
- S61 pad 1: Net-(D36-Pad2) -> Net-(D65-Pad2)
- S61 pad 2: Net-(R13-Pad2) -> Net-(R24-Pad2)
- S62 pad 1: Net-(D36-Pad2) -> Net-(D67-Pad2)
- S62 pad 2: Net-(R13-Pad2) -> Net-(R25-Pad2)
- S63 pad 1: Net-(D36-Pad2) -> Net-(D68-Pad2)
- S63 pad 2: Net-(R13-Pad2) -> Net-(R25-Pad2)
- S64 pad 1: Net-(D36-Pad2) -> Net-(D69-Pad2)
- S64 pad 2: Net-(R13-Pad2) -> Net-(R25-Pad2)
- S65 pad 1: Net-(D36-Pad2) -> Net-(D70-Pad2)
- S65 pad 2: Net-(R13-Pad2) -> Net-(R25-Pad2)
- S66 pad 1: Net-(D36-Pad2) -> Net-(D71-Pad2)
- S66 pad 2: Net-(R13-Pad2) -> Net-(R25-Pad2)
- S67 pad 1: Net-(D36-Pad2) -> Net-(D72-Pad2)
- S67 pad 2: Net-(R13-Pad2) -> Net-(R26-Pad2)
- S68 pad 1: Net-(D36-Pad2) -> Net-(D73-Pad2)
- S68 pad 2: Net-(R13-Pad2) -> Net-(R26-Pad2)
- S69 pad 1: Net-(D36-Pad2) -> Net-(D74-Pad2)
- S69 pad 2: Net-(R13-Pad2) -> Net-(R26-Pad2)
- S70 pad 1: Net-(D36-Pad2) -> Net-(D75-Pad2)
- S70 pad 2: Net-(R13-Pad2) -> Net-(R26-Pad2)
Routing:
- net Net-(D36-Pad2): track 118.1 -> 3.58 mm
- net Net-(D61-Pad2): track 0.00 -> 3.58 mm
- net Net-(D65-Pad2): track 0.00 -> 3.58 mm
- net Net-(D64-Pad2): track 0.00 -> 3.58 mm
- net Net-(D63-Pad2): track 0.00 -> 3.58 mm
- net Net-(D62-Pad2): track 0.00 -> 3.58 mm
- net Net-(D75-Pad2): track 0.00 -> 3.58 mm
- net Net-(D73-Pad2): track 0.00 -> 3.58 mm
- net Net-(D68-Pad2): track 0.00 -> 3.58 mm
- net Net-(D56-Pad2): track 0.00 -> 3.58 mm
- net Net-(D46-Pad2): track 0.00 -> 3.58 mm
- net Net-(D40-Pad2): track 0.00 -> 3.58 mm
- net Net-(D74-Pad2): track 0.00 -> 3.58 mm
- net Net-(D72-Pad2): track 0.00 -> 3.58 mm
- net Net-(D71-Pad2): track 0.00 -> 3.58 mm
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
Commit message: test points and current-limiting resistors placed
Parts:
- moved TP32 177.1 mm to (486.3, 189.9)
- moved TP29 174.2 mm to (464.5, 159.9)
- moved TP35 168.9 mm to (477.2, 265.8)
- moved TP28 165.9 mm to (457.9, 159.9)
- moved TP31 156.1 mm to (486.3, 170.6)
- moved TP34 153.8 mm to (486.3, 237.6)
- moved TP33 152.6 mm to (486.3, 208.7)
- moved TP36 128.5 mm to (331.4, 328.3)
- moved TP27 123.7 mm to (431.5, 166.8)
- moved TP38 108.4 mm to (331.4, 309.0)
- moved TP26 105.7 mm to (420.6, 161.2)
- moved TP25 103.3 mm to (401.8, 159.1)
- moved TP37 101.8 mm to (331.4, 319.4)
- moved R20 101.4 mm to (425.4, 161.2), turned to 270 degrees
- moved R16 100.7 mm to (347.9, 269.1)
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
Commit message: left mostly routed; kicad 6; need to cleanup files...
Parts:
- removed X1: ENCODER_ANO, Rotary_Encoder:ENCODER_ANO
- added J9: Conn_02x04_Top_Bottom, Connector_PinHeader_2.54mm:PinHeader_2x04_P2.54mm_Vertical, F.Cu at (178.4, 289.6)
- C1, C14, C15, C2, D1, D66, F1, F2, FB1, FB2, R7, U2, U3: moved to B.Cu
- J4, JP1: moved to F.Cu
- moved J7 179.5 mm to (477.3, 279.7), turned to 180 degrees
- moved C13 155.7 mm to (415.1, 273.3), turned to -90 degrees
- moved SW3 154.7 mm to (418.3, 275.5)
- moved SW4 154.7 mm to (419.4, 282.7)
- moved R23 153.2 mm to (428.1, 293.0), turned to 180 degrees
- moved C20 151.7 mm to (456.6, 273.9)
- moved C21 151.7 mm to (454.6, 281.1)
- moved C22 151.7 mm to (454.6, 279.6)
- moved U4 151.7 mm to (461.4, 278.4)
- moved C12 151.7 mm to (461.5, 287.0)
- moved C16 151.7 mm to (466.3, 284.4)
- moved C17 151.7 mm to (466.9, 273.0)
- moved C18 151.7 mm to (466.3, 282.9)
- moved C19 151.7 mm to (466.9, 274.5)
- moved C11 151.7 mm to (459.4, 287.0)
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Connections:
- net ~RST renamed ~{RST}
- D29 pad 1: L_ROW1 -> L_ROW5
- D30 pad 1: L_ROW2 -> L_ROW4
- J1 pad 4: Net-(J1-Pad4) -> unconnected-(J1-Pad4)
- J1 pad 6: Net-(J1-Pad6) -> unconnected-(J1-Pad6)
- J2 pad 1: +3V3 -> GND
- J2 pad 2: L_RX -> L_TX
- J2 pad 3: L_TX -> L_RX
- J2 pad 4: GND -> +3V3
- J3 pad 1: +3V3 -> GND
- J3 pad 2: L_SWDIO -> L_SWCLK
- J3 pad 3: L_SWCLK -> L_SWDIO
- J3 pad 4: GND -> +3V3
- J8 pad 4: Net-(J8-Pad4) -> unconnected-(J8-Pad4)
- J8 pad 6: Net-(J8-Pad6) -> unconnected-(J8-Pad6)
- S34 pad C: Net-(S34-PadC) -> unconnected-(S34-PadC)
- S34 pad D: Net-(S34-PadD) -> unconnected-(S34-PadD)
- SW2 pad 10: L_OPT4 -> L_OPT1
- SW2 pad 7: L_OPT1 -> L_OPT4
- SW2 pad 8: L_OPT2 -> L_OPT3
- SW2 pad 9: L_OPT3 -> L_OPT2
- TP15 pad 1: L_ENC_A -> ENC_A
- TP16 pad 1: L_ENC_B -> ENC_B
- TP17 pad 1: L_ENC_BN -> ENC_BN
- TP18 pad 1: L_ENC_DN -> ENC_DN
- TP19 pad 1: L_ENC_RT -> ENC_RT
- TP20 pad 1: L_ENC_UP -> ENC_UP
- TP21 pad 1: L_ENC_LF -> ENC_LF
- U1 pad 14: Net-(U1-Pad14) -> unconnected-(U1-Pad14)
- U1 pad 16: L_ENC_A -> ENC_B
- U1 pad 17: L_ENC_B -> ENC_A
- U1 pad 18: L_ROW1 -> ENC_LF
- U1 pad 19: L_ROW2 -> ENC_DN
- U1 pad 2: Net-(U1-Pad2) -> unconnected-(U1-Pad2)
- U1 pad 20: L_ROW3 -> ENC_RT
- U1 pad 21: L_ROW4 -> ENC_UP
- U1 pad 22: L_ROW5 -> ENC_BN
- U1 pad 3: Net-(U1-Pad3) -> unconnected-(U1-Pad3)
- U1 pad 38: L_ENC_BN -> L_ROW1
- U1 pad 39: L_ENC_DN -> L_ROW2
- U1 pad 4: Net-(U1-Pad4) -> unconnected-(U1-Pad4)
- U1 pad 40: L_ENC_RT -> L_ROW3
- U1 pad 41: L_ENC_UP -> L_ROW4
- U1 pad 45: L_ENC_LF -> L_ROW5
- U1 pad 5: Net-(U1-Pad5) -> unconnected-(U1-Pad5)
- U1 pad 6: Net-(U1-Pad6) -> unconnected-(U1-Pad6)
- U4 pad 14: Net-(U4-Pad14) -> unconnected-(U4-Pad14)
- U4 pad 2: Net-(U4-Pad2) -> unconnected-(U4-Pad2)
- U4 pad 3: Net-(U4-Pad3) -> unconnected-(U4-Pad3)
- U4 pad 4: Net-(U4-Pad4) -> unconnected-(U4-Pad4)
- U4 pad 45: Net-(U4-Pad45) -> unconnected-(U4-Pad45)
- U4 pad 5: Net-(U4-Pad5) -> unconnected-(U4-Pad5)
- U4 pad 6: Net-(U4-Pad6) -> unconnected-(U4-Pad6)
Routing:
- net L_ROW3: track 0.00 -> 302.1 mm, vias 0 -> 4
- net L_ROW5: track 0.00 -> 290.6 mm
- net L_ROW4: track 0.00 -> 276.8 mm, vias 0 -> 2
- net L_COL8: track 0.00 -> 163.3 mm, vias 0 -> 2
- net L_ROW2: track 0.00 -> 163.0 mm
- net +5V: track 0.00 -> 136.3 mm, vias 0 -> 2
- net L_ROW1: track 0.00 -> 119.5 mm
- net ~{RST}: track 0.00 -> 110.1 mm, vias 0 -> 1
- net Net-(R3-Pad2): track 0.00 -> 91.5 mm
- net Net-(R8-Pad2): track 0.00 -> 80.8 mm
- net Net-(R9-Pad2): track 0.00 -> 80.7 mm
- net Net-(R10-Pad2): track 0.00 -> 80.7 mm
- net Net-(R5-Pad2): track 0.00 -> 80.6 mm
- net Net-(R6-Pad2): track 0.00 -> 80.5 mm
- net Net-(R11-Pad2): track 0.00 -> 68.6 mm
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Other:
- net class Default removed
- net class Power removed
- board text added: "For Personal Use Only."
- board text added: "SOLIDWORKS Maker Product."

Commit message: more routing
Parts:
- moved C2 21.8 mm to (95.2, 160.7)
- moved D2 19.9 mm to (92.5, 155.6)
- moved R4 19.9 mm to (87.4, 155.6)
- moved U2 18.9 mm to (99.5, 155.6)
- moved C1 18.9 mm to (100.8, 160.7)
- moved D1 17.3 mm to (107.3, 151.1), turned to 180 degrees
- moved FB1 17.1 mm to (107.3, 154.9)
- moved F1 13.0 mm to (108.0, 146.1), turned to 180 degrees
- moved TP5 8.98 mm to (166.4, 156.8)
- moved TP4 5.85 mm to (182.9, 157.5)
- moved R7 1.91 mm to (153.7, 144.1), turned to 90 degrees
- moved J3 0.64 mm to (186.7, 150.5)
- moved R1 0.64 mm to (113.7, 146.7)
- moved TP14 0.64 mm to (84.5, 262.3)
- moved J2 0.63 mm to (191.1, 153.0)
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Routing:
- net +3V3: track 52.0 -> 198.9 mm
- net L_COL7: track 4.29 -> 72.4 mm
- net L_USB_D+: track 0.00 -> 67.1 mm, vias 0 -> 2
- net L_USB_D-: track 0.00 -> 66.3 mm, vias 0 -> 2
- net L_COL1: track 4.81 -> 58.0 mm, vias 1 -> 2
- net L_COL6: track 4.57 -> 57.5 mm
- net L_COL5: track 4.49 -> 39.1 mm
- net L_COL2: track 4.98 -> 38.7 mm, vias 1 -> 2
- net ENC_B: track 8.67 -> 26.2 mm, vias 0 -> 1
- net ENC_A: track 7.62 -> 23.3 mm, vias 0 -> 1
- net L_COL3: track 4.30 -> 19.8 mm, vias 1 -> 2
- net ENC_LF: track 7.62 -> 21.5 mm, vias 0 -> 1
- net ENC_DN: track 9.72 -> 21.7 mm, vias 0 -> 1
- net +5V: track 136.3 -> 146.5 mm
- net ENC_RT: track 8.67 -> 18.9 mm, vias 0 -> 1
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