File: thumbler.kicad_sch (KiCad schematic)
At the start: 257 parts, among them J1 USB_B_Micro, J2 Conn_01x04, J3 Conn_01x04, J4 DIN-5_180degree, J5 Conn_01x04, J6 DIN-5_180degree, J7 Conn_01x04, J8 USB_B_Micro, J9 Conn_02x04_Top_Bottom, SW1 SW_Push, SW2 SW_DIP_x05, SW3 SW_Push, SW4 SW_DIP_x05, U1 STM32F072C8Tx, U2 MCP1700-3302E_SOT89, U3 MCP1700-3302E_SOT89, U4 STM32F072C8Tx

Commit message: more routing
Connections:
- net L_ROW1: no longer D29.1 (K)
- net L_ROW2: no longer D30.1 (K)
- net L_ROW4: now also D30.1 (K)
- net L_ROW5: now also D29.1 (K)
Changed lines of the file:
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@@
   (global_label "L_ROW3" (shape input) (at 267.97 292.1 0) (fields_autoplaced)
     (effects (font (size 1.27 1.27)) (justify left))
-    (property "Intersheet References" "${INTERSHEET_REFS}" (id 0) (at 0 0 0)
-      (effects (font (size 1.27 1.27)) hide)
+    (property "Intersheet References" "${INTERSHEET_REFS}" (id 0) (at 277.5513 292.0206 0)
+      (effects (font (size 1.27 1.27)) (justify left) hide)
     )
   )
@@
     )
   )
-  (global_label "L_ROW2" (shape input) (at 267.97 280.67 0) (fields_autoplaced)
-    (effects (font (size 1.27 1.27)) (justify left))
-    (property "Intersheet References" "${INTERSHEET_REFS}" (id 0) (at 0 0 0)
-      (effects (font (size 1.27 1.27)) hide)
+  (global_label "L_ROW4" (shape input) (at 267.97 280.67 0) (fields_autoplaced)
+    (effects (font (size 1.27 1.27)) (justify left))
+    (property "Intersheet References" "${INTERSHEET_REFS}" (id 0) (at 277.5513 280.5906 0)
+      (effects (font (size 1.27 1.27)) (justify left) hide)
     )
   )
@@
     )
   )
-  (global_label "L_ROW1" (shape input) (at 267.97 269.24 0) (fields_autoplaced)
-    (effects (font (size 1.27 1.27)) (justify left))
-    (property "Intersheet References" "${INTERSHEET_REFS}" (id 0) (at 0 0 0)
-      (effects (font (size 1.27 1.27)) hide)
-    )
-  )
+  (global_label "L_ROW5" (shape input) (at 267.97 269.24 0) (fields_autoplaced)
+    (effects (font (size 1.27 1.27)) (justify left))
+    (property "Intersheet References" "${INTERSHEET_REFS}" (id 0) (at 277.5513 269.1606 0)
+      (effects (font (size 1.27 1.27)) (justify left) hide)
+    )
+  )
