File: left/thumbler_left.kicad_pcb (KiCad board)
At the start: 4 copper layers, 187.8 x 203.6 mm, 132 parts, among them J1 USB_B_Micro, J2 Conn_01x04, J3 Conn_01x04, J4 DIN-5_180degree, J9 Conn_02x04_Top_Bottom, SW1 SW_Push, SW2 SW_DIP_x05, U1 STM32F072C8Tx, U2 MCP1700-3302E_SOT89

Commit message: ready to manufacture?
Parts:
- moved TP1 1.89 mm to (123.2, 141.5)
Changed lines of the file:
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@@
   )
   (footprint "TestPoint:TestPoint_Pad_D2.0mm" (layer "F.Cu")
-    (at 123.825 139.7)
+    (at 123.19 141.478)
     (descr "SMD pad as test Point, diameter 2.0mm")
     (tags "test point SMD pad")
@@
     (property "Sheetname" "")
     (attr exclude_from_pos_files)
-    (fp_text reference "TP1" (at 0 2.286) (layer "F.SilkS")
+    (fp_text reference "TP1" (at 0 -2.032) (layer "F.SilkS")
       (effects (font (size 1 1) (thickness 0.15)))
     )
@@
     (effects (font (size 1 1) (thickness 0.15)))
   )
+  (gr_text "5V" (at 123.19 143.764) (layer "F.SilkS")
+    (effects (font (size 1 1) (thickness 0.15)))
+  )
   (gr_text "A" (at 165.735 292.1 270) (layer "F.SilkS")
     (effects (font (size 1 1) (thickness 0.15)))
@@
   (segment (start 145.811 176.0322) (end 135.811 186.0322) (width 0.25) (layer "F.Cu") (net 43))
   (segment (start 102.3248 186.0322) (end 102.29 186.067) (width 0.25) (layer "F.Cu") (net 43))
-  (segment (start 123.825 139.7) (end 123.825 151.765) (width 0.35) (layer "F.Cu") (net 44))
-  (segment (start 123.825 139.7) (end 124.825 138.7) (width 0.35) (layer "F.Cu") (net 44))
-  (segment (start 216.240831 152.232831) (end 219.817306 152.232831) (width 0.35) (layer "F.Cu") (net 44))
-  (segment (start 124.825 138.7) (end 202.708 138.7) (width 0.35) (layer "F.Cu") (net 44))
-  (segment (start 202.708 138.7) (end 216.240831 152.232831) (width 0.35) (layer "F.Cu") (net 44))
-  (via (at 123.825 151.765) (size 0.6) (drill 0.3) (layers "F.Cu" "B.Cu") (net 44))
+  (segment (start 124.825 138.7) (end 123.19 140.335) (width 0.35) (layer "F.Cu") (net 44))
+  (segment (start 123.19 140.335) (end 123.19 151.765) (width 0.35) (layer "F.Cu") (net 44))
+  (segment (start 219.817306 152.232831) (end 216.240831 152.232831) (width 0.35) (layer "F.Cu") (net 44))
+  (segment (start 216.240831 152.232831) (end 202.708 138.7) (width 0.35) (layer "F.Cu") (net 44))
+  (segment (start 202.708 138.7) (end 124.825 138.7) (width 0.35) (layer "F.Cu") (net 44))
+  (via (at 123.19 151.765) (size 0.6) (drill 0.3) (layers "F.Cu" "B.Cu") (net 44))
+  (segment (start 122.3 153.67) (end 123.19 152.78) (width 0.35) (layer "B.Cu") (net 44))
   (segment (start 117.085 155.575) (end 120.395 155.575) (width 0.35) (layer "B.Cu") (net 44))
-  (segment (start 123.825 152.145) (end 123.825 151.765) (width 0.35) (layer "B.Cu") (net 44))
+  (segment (start 123.19 152.78) (end 123.19 151.765) (width 0.35) (layer "B.Cu") (net 44))
   (segment (start 120.395 155.575) (end 122.3 153.67) (width 0.35) (layer "B.Cu") (net 44))
   (segment (start 114.935 153.425) (end 117.085 155.575) (width 0.35) (layer "B.Cu") (net 44))
-  (segment (start 122.3 153.67) (end 123.825 152.145) (width 0.35) (layer "B.Cu") (net 44))
   (segment (start 173.7075 146.935) (end 174.756 146.935) (width 0.25) (layer "F.Cu") (net 45))
   (segment (start 174.756 146.935) (end 175.006 146.685) (width 0.25) (layer "F.Cu") (net 45))
