File: right/thumbler_right.kicad_pcb (KiCad board)
At the start: 4 copper layers, 187.8 x 203.6 mm, 143 parts, among them J5 Conn_01x04, J6 DIN-5_180degree, J7 Conn_01x04, J8 USB_B_Micro, SW3 SW_Push, SW4 SW_DIP_x05, U3 MCP1700-3302E_SOT89, U4 STM32F072C8Tx

Commit message: ready to manufacture?
Parts:
- moved TP22 5.14 mm to (436.4, 140.7)
- moved TP30 1.51 mm to (361.4, 242.3)
- moved TP23 1.21 mm to (359.9, 163.5)
- moved R20 1.02 mm to (423.7, 158.8)
- moved R16 0.75 mm to (361.4, 246.9)
- moved D45 0.38 mm to (420.6, 145.0)
- moved D51 0.38 mm to (415.5, 145.0)
- moved D55 0.38 mm to (410.5, 145.0)
- moved R14 0.25 mm to (420.6, 140.2)
- moved R17 0.25 mm to (415.5, 140.2)
- moved R18 0.25 mm to (410.5, 140.2)
- moved J6 0.09 mm to (343.6, 139.2)
- moved TP26 0.05 mm to (419.4, 157.9)
Routing:
- net +5V: track 130.0 -> 126.4 mm
- net R_COL1: track 48.0 -> 45.5 mm
- net R_COL4: track 28.9 -> 29.9 mm
- net Net-(R20-Pad2): track 80.0 -> 80.9 mm
- net R_COL8: track 158.9 -> 159.7 mm
- net Net-(R16-Pad2): track 71.6 -> 72.3 mm
- net R_ROW5: track 342.5 -> 343.2 mm
Other:
- board text added: "3V3"
- board text added: "5V"
- board text added: "CLK"
- board text added: "COL1"
- board text added: "COL2"
- board text added: "COL3"
- board text added: "COL4"
- board text added: "COL5"
- board text added: "COL6"
- board text added: "COL7"
- board text added: "COL8"
- board text added: "GND"
- board text added: "IO"
- board text added: "JLCJLCJLCJLC"
- board text added: "ROW1"
- board text added: "ROW2"
- board text added: "ROW3"
- board text added: "ROW4"
- board text added: "ROW5"
- board text added: "RST"
- board text added: "RX"
- board text added: "TX"
