File: right/thumbler_right.kicad_sch (KiCad schematic)
At the start: 143 parts, among them J5 Conn_01x04, J6 DIN-5_180degree, J7 Conn_01x04, J8 USB_B_Micro, SW3 SW_Push, SW4 SW_DIP_x05, U3 MCP1700-3302E_SOT89, U4 STM32F072C8Tx

Commit message: ready to manufacture?
Parts:
- renumbered H1 to H?, H6 to H?, H5 to H?, H3 to H?, H7 to H?, H4 to H?, H2 to H?
Changed lines of the file:
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@@
   (no_connect (at 407.67 196.85))
   (no_connect (at 374.65 153.67))
-  (bus_entry (at 341.63 240.03) (size 2.54 2.54)
-    (stroke (width 0) (type default) (color 0 0 0 0))
-  )
-  (bus_entry (at 354.33 261.62) (size 2.54 2.54)
-    (stroke (width 0) (type default) (color 0 0 0 0))
-  )
   (bus_entry (at 201.93 242.57) (size 2.54 2.54)
     (stroke (width 0) (type default) (color 0 0 0 0))
@@
   (symbol (lib_id "Mechanical:MountingHole") (at 295.91 222.25 0) (unit 1)
     (in_bom yes) (on_board yes) (fields_autoplaced)
-    (property "Reference" "H1" (id 0) (at 298.45 220.9799 0)
+    (property "Reference" "H?" (id 0) (at 298.45 220.9799 0)
       (effects (font (size 1.27 1.27)) (justify left))
     )
@@
   (symbol (lib_id "Mechanical:MountingHole") (at 295.91 260.35 0) (unit 1)
     (in_bom yes) (on_board yes) (fields_autoplaced)
-    (property "Reference" "H6" (id 0) (at 298.45 259.0799 0)
+    (property "Reference" "H?" (id 0) (at 298.45 259.0799 0)
       (effects (font (size 1.27 1.27)) (justify left))
     )
@@
   (symbol (lib_id "Mechanical:MountingHole") (at 295.91 252.73 0) (unit 1)
     (in_bom yes) (on_board yes) (fields_autoplaced)
-    (property "Reference" "H5" (id 0) (at 298.45 251.4599 0)
+    (property "Reference" "H?" (id 0) (at 298.45 251.4599 0)
       (effects (font (size 1.27 1.27)) (justify left))
     )
@@
   (symbol (lib_id "Mechanical:MountingHole") (at 295.91 237.49 0) (unit 1)
     (in_bom yes) (on_board yes) (fields_autoplaced)
-    (property "Reference" "H3" (id 0) (at 298.45 236.2199 0)
+    (property "Reference" "H?" (id 0) (at 298.45 236.2199 0)
       (effects (font (size 1.27 1.27)) (justify left))
     )
@@
   (symbol (lib_id "Mechanical:MountingHole") (at 295.91 267.97 0) (unit 1)
     (in_bom yes) (on_board yes) (fields_autoplaced)
-    (property "Reference" "H7" (id 0) (at 298.45 266.6999 0)
+    (property "Reference" "H?" (id 0) (at 298.45 266.6999 0)
       (effects (font (size 1.27 1.27)) (justify left))
     )
@@
   (symbol (lib_id "Mechanical:MountingHole") (at 295.91 245.11 0) (unit 1)
     (in_bom yes) (on_board yes)
-    (property "Reference" "H4" (id 0) (at 298.45 243.8399 0)
+    (property "Reference" "H?" (id 0) (at 298.45 243.8399 0)
       (effects (font (size 1.27 1.27)) (justify left))
     )
@@
   (symbol (lib_id "Mechanical:MountingHole") (at 295.91 229.87 0) (unit 1)
     (in_bom yes) (on_board yes) (fields_autoplaced)
-    (property "Reference" "H2" (id 0) (at 298.45 228.5999 0)
+    (property "Reference" "H?" (id 0) (at 298.45 228.5999 0)
       (effects (font (size 1.27 1.27)) (justify left))
     )
@@
     )
     (path "/3a4f9df2-ba54-4885-acb5-b932e70c7f8c"
-      (reference "H1") (unit 1) (value "MountingHole") (footprint "MountingHole:MountingHole_3.2mm_M3")
-    )
-    (path "/fadf0793-28c7-4aff-87f6-cd927bf2c7ed"
-      (reference "H2") (unit 1) (value "MountingHole") (footprint "MountingHole:MountingHole_3.2mm_M3")
-    )
-    (path "/be87df51-465c-4021-9022-67bf1bd3ebba"
-      (reference "H3") (unit 1) (value "MountingHole") (footprint "MountingHole:MountingHole_3.2mm_M3")
+      (reference "H?") (unit 1) (value "MountingHole") (footprint "MountingHole:MountingHole_3.2mm_M3")
     )
-    (path "/edf39b35-3beb-4e49-8949-c9e97e7cef96"
-      (reference "H4") (unit 1) (value "MountingHole") (footprint "MountingHole:MountingHole_3.2mm_M3")
+    (path "/749344f6-c4bf-4a93-9320-7fb13f6d1d28"
+      (reference "H?") (unit 1) (value "MountingHole") (footprint "MountingHole:MountingHole_3.2mm_M3")
     )
     (path "/a5528b7d-5c94-42cc-b826-5176581d130a"
-      (reference "H5") (unit 1) (value "MountingHole") (footprint "MountingHole:MountingHole_3.2mm_M3")
+      (reference "H?") (unit 1) (value "MountingHole") (footprint "MountingHole:MountingHole_3.2mm_M3")
     )
-    (path "/749344f6-c4bf-4a93-9320-7fb13f6d1d28"
-      (reference "H6") (unit 1) (value "MountingHole") (footprint "MountingHole:MountingHole_3.2mm_M3")
+    (path "/be87df51-465c-4021-9022-67bf1bd3ebba"
+      (reference "H?") (unit 1) (value "MountingHole") (footprint "MountingHole:MountingHole_3.2mm_M3")
     )
     (path "/e745904e-442e-4cb4-937c-49c360e59543"
-      (reference "H7") (unit 1) (value "MountingHole") (footprint "MountingHole:MountingHole_3.2mm_M3")
+      (reference "H?") (unit 1) (value "MountingHole") (footprint "MountingHole:MountingHole_3.2mm_M3")
+    )
+    (path "/edf39b35-3beb-4e49-8949-c9e97e7cef96"
+      (reference "H?") (unit 1) (value "MountingHole") (footprint "MountingHole:MountingHole_3.2mm_M3")
+    )
+    (path "/fadf0793-28c7-4aff-87f6-cd927bf2c7ed"
+      (reference "H?") (unit 1) (value "MountingHole") (footprint "MountingHole:MountingHole_3.2mm_M3")
     )
     (path "/00000000-0000-0000-0000-000064abcecf"
